File: Processing_and_measuring/Processing_and_measuring.kicad_sch (KiCad schematic)
At the start: 37 parts, among them J1 Conn_02x07_Counter_Clockwise, J2 Conn_01x02_Pin, J3 Conn_02x07_Counter_Clockwise, U1 TPL7407LAD, U2 CD74HC4067M, U3 AVR128DA48x-xPT, U4 TPL7407LAD, Y1 X_Crystal_16MHz_18pF

Commit message: Layout work and power
Connections:
- net Power: now also A1.8 (VMOT)
Changed lines of the file:
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@@
+	(global_label "Power"
+		(shape input)
+		(at 64.77 138.43 90)
+		(fields_autoplaced yes)
+		(effects
+			(font
+				(size 1.27 1.27)
+			)
+			(justify left)
+		)
+		(property "Intersheetrefs" "${INTERSHEET_REFS}"
+			(at 64.77 129.8205 90)
+			(effects
+				(font
+					(size 1.27 1.27)
+				)
+				(justify left)
+				(hide yes)
+			)
+		)
+	)
 	(global_label "Power"
 		(shape input)
