File: Processing_and_measuring/_autosave-Processing_and_measuring.kicad_pcb (KiCad board)
At the start: 2 copper layers, 49 parts, among them J1 Conn_02x07_Counter_Clockwise, J2 Conn_01x02_Pin, J3 Conn_02x07_Counter_Clockwise, J4 Conn_01x04_Pin, J5 Conn_01x02_Pin, J6 Conn_01x02_Pin, U1 TPL7407LAD, U2 CD74HC4067M, U3 AVR128DA48x-xPT, U4 TPL7407LAD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

Commit message: Buck converter layout mostly
Parts:
- removed J5: Conn_01x02_Pin, Connector_PinHeader_1.00mm:PinHeader_1x02_P1.00mm_Horizontal
- moved C3 57.9 mm to (168.5, 72.0)
- moved R18 5.43 mm to (172.7, 65.5), turned to 0 degrees
- moved C4 4.64 mm to (171.9, 67.9), turned to 90 degrees
- moved R20 1.99 mm to (175.2, 67.9), turned to 90 degrees
- moved R17 0.67 mm to (173.6, 67.9), turned to 90 degrees
- turned C5 to 0 degrees
Connections:
- J2 pad 2: VIN -> Power
Routing:
- net +5V: track 65.5 -> 75.4 mm
- net GND: track 31.0 -> 39.7 mm, vias 9 -> 10
- net Net-(VR1-EN): track 5.55 -> 10.2 mm, vias 0 -> 2
- net Net-(VR1-FB): track 2.76 -> 5.35 mm
